File: ventilatorcontrol/hardwareadapters/ventilatorconnectors/AudioJackMotorController/MotorController.brd (EAGLE design)
At the start: 50.8 x 80 mm, 20 parts, among them J1 39-30-1060, J2 39-30-1060, X2 1503_10

Commit message: updated hardware files with newer circuit
Parts:
- R1: value 10k -> 27k
- R3: value 10k -> 560k
- R4: value 10k -> 4.7k
- moved R1 31.9 mm to (29.8, 51.8), turned to 270 degrees
- moved R2 2.56 mm to (15.9, 22.2)
Connections:
- new net N$5: SIGNAL_AMP_.6, SIGNAL_AMP_.7
- net GND: no longer SIGNAL_AMP_.6
- net N$1: no longer R1.1
- net N$4: now also R1.1
Routing:
- net N$1: track 20.8 -> 16.1 mm
- net N$4: track 13.1 -> 15.9 mm
- net N$5: track 0.00 -> 2.54 mm
Changed lines of the file:
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@@
 <grid distance="12.5" unitdist="mil" unit="mil" style="lines" multiple="1" display="no" altdistance="5" altunitdist="mil" altunit="mil"/>
 <layers>
-<layer number="1" name="Top" color="4" fill="1" visible="no" active="yes"/>
+<layer number="1" name="Top" color="4" fill="1" visible="yes" active="yes"/>
 <layer number="16" name="Bottom" color="1" fill="1" visible="yes" active="yes"/>
 <layer number="17" name="Pads" color="2" fill="1" visible="yes" active="yes"/>
@@
 <attribute name="VALUE" x="35.55243125" y="56.96985" size="1.78153125" layer="27" ratio="10" rot="R270"/>
 </element>
-<element name="R1" library="rcl" library_urn="urn:adsk.eagle:library:334" package="0204/7" package3d_urn="urn:adsk.eagle:package:23498/2" value="10k" x="15.5575" y="23.1775" smashed="yes" rot="R180">
-<attribute name="NAME" x="12.7" y="25.3746" size="0.9906" layer="25" ratio="10" rot="R180"/>
-<attribute name="POPULARITY" value="79" x="-7.3025" y="76.5175" size="1.778" layer="27" rot="R180" display="off"/>
-<attribute name="SPICEPREFIX" value="R" x="-7.3025" y="76.5175" size="1.778" layer="27" rot="R180" display="off"/>
-<attribute name="VALUE" x="17.1831" y="23.6601" size="0.9906" layer="27" ratio="10" rot="R180"/>
-</element>
-<element name="R2" library="rcl" library_urn="urn:adsk.eagle:library:334" package="0204/7" package3d_urn="urn:adsk.eagle:package:23498/2" value="10k" x="15.5575" y="19.685" smashed="yes">
-<attribute name="NAME" x="11.1125" y="20.9804" size="0.9906" layer="25" ratio="10"/>
-<attribute name="POPULARITY" value="79" x="48.5775" y="-33.655" size="1.778" layer="27" display="off"/>
-<attribute name="SPICEPREFIX" value="R" x="48.5775" y="-33.655" size="1.778" layer="27" display="off"/>
-<attribute name="VALUE" x="13.9319" y="19.2024" size="0.9906" layer="27" ratio="10"/>
-</element>
-<element name="R3" library="rcl" library_urn="urn:adsk.eagle:library:334" package="0204/7" package3d_urn="urn:adsk.eagle:package:23498/2" value="10k" x="31.4325" y="18.415" smashed="yes">
+<element name="R1" library="rcl" library_urn="urn:adsk.eagle:library:334" package="0204/7" package3d_urn="urn:adsk.eagle:package:23498/2" value="27k" x="29.845" y="51.7525" smashed="yes" rot="R270">
+<attribute name="NAME" x="27.6479" y="48.895" size="0.9906" layer="25" ratio="10" rot="R270"/>
+<attribute name="POPULARITY" value="79" x="-23.495" y="28.8925" size="1.778" layer="27" rot="R270" display="off"/>
+<attribute name="SPICEPREFIX" value="R" x="-23.495" y="28.8925" size="1.778" layer="27" rot="R270" display="off"/>
+<attribute name="VALUE" x="29.3624" y="53.3781" size="0.9906" layer="27" ratio="10" rot="R270"/>
+</element>
+<element name="R2" library="rcl" library_urn="urn:adsk.eagle:library:334" package="0204/7" package3d_urn="urn:adsk.eagle:package:23498/2" value="10k" x="15.875" y="22.225" smashed="yes">
+<attribute name="NAME" x="11.43" y="23.5204" size="0.9906" layer="25" ratio="10"/>
+<attribute name="POPULARITY" value="79" x="48.895" y="-31.115" size="1.778" layer="27" display="off"/>
+<attribute name="SPICEPREFIX" value="R" x="48.895" y="-31.115" size="1.778" layer="27" display="off"/>
+<attribute name="VALUE" x="14.2494" y="21.7424" size="0.9906" layer="27" ratio="10"/>
+</element>
+<element name="R3" library="rcl" library_urn="urn:adsk.eagle:library:334" package="0204/7" package3d_urn="urn:adsk.eagle:package:23498/2" value="560k" x="31.4325" y="18.415" smashed="yes">
 <attribute name="NAME" x="27.305" y="19.7104" size="0.9906" layer="25" ratio="10"/>
 <attribute name="POPULARITY" value="79" x="74.6125" y="-34.925" size="1.778" layer="27" display="off"/>
@@
 <attribute name="VALUE" x="29.8069" y="17.9324" size="0.9906" layer="27" ratio="10"/>
 </element>
-<element name="R4" library="rcl" library_urn="urn:adsk.eagle:library:334" package="0204/7" package3d_urn="urn:adsk.eagle:package:23498/2" value="10k" x="31.4325" y="14.9225" smashed="yes">
+<element name="R4" library="rcl" library_urn="urn:adsk.eagle:library:334" package="0204/7" package3d_urn="urn:adsk.eagle:package:23498/2" value="4.7k" x="31.4325" y="14.9225" smashed="yes">
 <attribute name="NAME" x="26.9875" y="16.2179" size="0.9906" layer="25" ratio="10"/>
 <attribute name="POPULARITY" value="79" x="84.7725" y="-38.4175" size="1.778" layer="27" display="off"/>
@@
 <signal name="N$1" class="2">
 <contactref element="SIGNAL_AMP_" pad="3"/>
-<contactref element="R1" pad="1"/>
 <contactref element="R2" pad="2"/>
 <contactref element="C5" pad="+"/>
-<wire x1="16.8275" y1="28.8925" x2="16.8275" y2="24.4475" width="0.889" layer="16"/>
-<wire x1="16.8275" y1="24.4475" x2="18.0975" y2="23.1775" width="0.889" layer="16"/>
-<wire x1="18.0975" y1="23.1775" x2="19.3675" y2="23.1775" width="0.889" layer="16"/>
-<wire x1="19.3675" y1="19.685" x2="19.3675" y2="23.1775" width="0.889" layer="16"/>
-<wire x1="27.6225" y1="26.3525" x2="22.225" y2="26.3525" width="0.889" layer="16"/>
-<wire x1="22.225" y1="26.3525" x2="19.3675" y2="23.495" width="0.889" layer="16"/>
-<wire x1="19.3675" y1="23.495" x2="19.3675" y2="23.1775" width="0.889" layer="16"/>
+<wire x1="16.8275" y1="28.8925" x2="19.3675" y2="26.3525" width="0.889" layer="16"/>
+<wire x1="19.3675" y1="26.3525" x2="27.6225" y2="26.3525" width="0.889" layer="16"/>
+<wire x1="19.685" y1="22.225" x2="19.685" y2="26.035" width="0.889" layer="16"/>
+<wire x1="19.685" y1="26.035" x2="19.3675" y2="26.3525" width="0.889" layer="16"/>
 </signal>
 <signal name="N$2" class="2">
@@
 <wire x1="32.7025" y1="55.5625" x2="29.21" y2="59.055" width="0.889" layer="16"/>
 <wire x1="29.21" y1="59.055" x2="29.21" y2="60.0075" width="0.889" layer="16"/>
+<contactref element="R1" pad="1"/>
+<wire x1="29.845" y1="55.5625" x2="32.7025" y2="55.5625" width="0.889" layer="16"/>
 </signal>
 <signal name="N$7" class="2">
@@
 <contactref element="R4" pad="1"/>
 <contactref element="SIGNAL_AMP_" pad="5"/>
-<contactref element="SIGNAL_AMP_" pad="6"/>
 <contactref element="SIGNAL_AMP_" pad="4"/>
 <contactref element="J1" pad="5"/>
@@
 <contactref element="X1" pad="2"/>
 </signal>
+<signal name="N$5">
+<contactref element="SIGNAL_AMP_" pad="6"/>
+<contactref element="SIGNAL_AMP_" pad="7"/>
+<wire x1="35.2425" y1="28.8925" x2="35.2425" y2="26.3525" width="0.889" layer="16"/>
+</signal>
 </signals>
